Commit message: fixed urdf bug

File: hri_hand_control/urdf/hj_hand.urdf.xacro (robot description, xacro)
@@ -37,5 +37,5 @@
             <collision>
                   <geometry>
-                        <mesh filename="package://hri_hand_control/urdf/F03_AL_link_hand_wrist_part.stl" scale="0.001 0.001 0.001"/>
+                        <mesh filename="package://hri_hand_control/urdf/mesh/F03_AL_link_hand_wrist_part.stl" scale="0.001 0.001 0.001"/>
                   </geometry>
                   <origin xyz = "0.0 0.0 0.0" rpy = "1.57 0.0 0.0"/>
@@ -58,5 +58,5 @@
             <visual>
                   <geometry>
-                  <mesh filename="package:/hri_hand_control/urdf/mesh/F03_AL_palm.stl" scale="0.001 0.001 0.001"/>
+                  <mesh filename="package://hri_hand_control/urdf/mesh/F03_AL_palm.stl" scale="0.001 0.001 0.001"/>
                   </geometry>
                   <origin xyz = "${hand_palm_x} ${hand_palm_y} ${hand_palm_z}" rpy = "${hand_palm_r} ${hand_palm_p} ${hand_palm_yaw}"/>
